File: Kicad/Aquautomatic_v1_1/zerocross_triacDrive_sch.kicad_sch (KiCad schematic)
At the start: 27 parts

Commit message: [Add anny files from KICAD folder]
- Add anny files from KICAD folder
Parts:
- C?: footprint (none) -> Capacitor_SMD:C_0805_2012Metric_Pad1.18x1.45mm_HandSolder
- R?: footprint (none) -> Resistor_SMD:R_1206_3216Metric_Pad1.30x1.75mm_HandSolder
Changed lines of the file:
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@@
     (property "Reference" "R?" (id 0) (at 95.25 55.88 90))
     (property "Value" "100K" (id 1) (at 95.25 58.42 90))
-    (property "Footprint" "" (id 2) (at 95.25 62.23 0)
+    (property "Footprint" "Resistor_SMD:R_1206_3216Metric_Pad1.30x1.75mm_HandSolder" (id 2) (at 95.25 62.23 0)
       (effects (font (size 1.27 1.27)) hide)
     )
@@
       (effects (font (size 1.27 1.27)) (justify left))
     )
-    (property "Footprint" "" (id 2) (at 105.41 71.12 0)
+    (property "Footprint" "Capacitor_SMD:C_0805_2012Metric_Pad1.18x1.45mm_HandSolder" (id 2) (at 105.41 71.12 0)
       (effects (font (size 1.27 1.27)) hide)
     )
